File: schematics/watchdog/w.sch (KiCad schematic (older format))
At the start: 18 parts, among them J1 VOUT 3V, J2 Power IN, J3 I2C, J4 VOUT 5V, Q1 IRF4905, Q2 2N2219, Q3 IRF4905, Q4 2N2219, U1 ATtiny85-20PU, U2 AMS1117

Commit message: Work in progress.
Parts:
- added J5: Conn_01x08_MountingPin, Connector_PinHeader_2.54mm:PinHeader_1x08_P2.54mm_Vertical, symbol Connector_Generic_MountingPin:Conn_01x08_MountingPin
- C1, C2: footprint (none) -> Capacitor_THT:CP_Axial_L10.0mm_D6.0mm_P15.00mm_Horizontal
- J1, J2, J3, J4: footprint (none) -> Connector_PinHeader_2.54mm:PinHeader_1x01_P2.54mm_Horizontal
- R1, R2, R3, R4, R5, R6: footprint (none) -> Resistor_THT:R_Axial_DIN0204_L3.6mm_D1.6mm_P1.90mm_Vertical
Connections:
- net +5V: now also J5.1 (Pin_1)
- net CLK: now also J5.7 (Pin_7)
- net DAT: now also J5.8 (Pin_8)
- net GND: now also J5.2 (Pin_2), J5.4 (Pin_4), J5.6 (Pin_6)
- net O3V: now also J5.5 (Pin_5)
- net O5V: now also J5.3 (Pin_3)
Changed lines of the file:
@@
 F 0 "J2" H 9656 3878 50  0000 C CNN
 F 1 "Power IN" H 9656 3787 50  0000 C CNN
-F 2 "" H 9550 3700 50  0001 C CNN
+F 2 "Connector_PinHeader_2.54mm:PinHeader_1x01_P2.54mm_Horizontal" H 9550 3700 50  0001 C CNN
 F 3 "~" H 9550 3700 50  0001 C CNN
 	1    9550 3700
@@
 L power:+5V #PWR0102
 U 1 1 606E46A9
-P 8900 3600
-F 0 "#PWR0102" H 8900 3450 50  0001 C CNN
-F 1 "+5V" H 8915 3773 50  0000 C CNN
-F 2 "" H 8900 3600 50  0001 C CNN
-F 3 "" H 8900 3600 50  0001 C CNN
-	1    8900 3600
+P 8800 3450
+F 0 "#PWR0102" H 8800 3300 50  0001 C CNN
+F 1 "+5V" H 8815 3623 50  0000 C CNN
+F 2 "" H 8800 3450 50  0001 C CNN
+F 3 "" H 8800 3450 50  0001 C CNN
+	1    8800 3450
 	0    -1   -1   0
 $EndComp
@@
 F 0 "J3" H 9656 3128 50  0000 C CNN
 F 1 "I2C" H 9656 3037 50  0000 C CNN
-F 2 "" H 9550 2950 50  0001 C CNN
+F 2 "Connector_PinHeader_2.54mm:PinHeader_1x01_P2.54mm_Horizontal" H 9550 2950 50  0001 C CNN
 F 3 "~" H 9550 2950 50  0001 C CNN
 	1    9550 2950
@@
 F 0 "J1" H 9656 4628 50  0000 C CNN
 F 1 "VOUT 3V" H 9656 4537 50  0000 C CNN
-F 2 "" H 9550 4450 50  0001 C CNN
+F 2 "Connector_PinHeader_2.54mm:PinHeader_1x01_P2.54mm_Horizontal" H 9550 4450 50  0001 C CNN
 F 3 "~" H 9550 4450 50  0001 C CNN
 	1    9550 4450
@@
 F 0 "J4" H 9606 2128 50  0000 C CNN
 F 1 "VOUT 5V" H 9606 2037 50  0000 C CNN
-F 2 "" H 9500 1950 50  0001 C CNN
+F 2 "Connector_PinHeader_2.54mm:PinHeader_1x01_P2.54mm_Horizontal" H 9500 1950 50  0001 C CNN
 F 3 "~" H 9500 1950 50  0001 C CNN
 	1    9500 1950
@@
 F 0 "R3" H 7170 4296 50  0000 L CNN
 F 1 "R" H 7170 4205 50  0000 L CNN
-F 2 "" V 7030 4250 50  0001 C CNN
+F 2 "Resistor_THT:R_Axial_DIN0204_L3.6mm_D1.6mm_P1.90mm_Vertical" V 7030 4250 50  0001 C CNN
 F 3 "~" H 7100 4250 50  0001 C CNN
 	1    7100 4250
@@
 F 0 "R1" V 6243 4600 50  0000 C CNN
 F 1 "R" V 6334 4600 50  0000 C CNN
-F 2 "" V 6380 4600 50  0001 C CNN
+F 2 "Resistor_THT:R_Axial_DIN0204_L3.6mm_D1.6mm_P1.90mm_Vertical" V 6380 4600 50  0001 C CNN
 F 3 "~" H 6450 4600 50  0001 C CNN
 	1    6450 4600
@@
 F 0 "R2" H 6770 4296 50  0000 L CNN
 F 1 "R" H 6770 4205 50  0000 L CNN
-F 2 "" V 6630 4250 50  0001 C CNN
+F 2 "Resistor_THT:R_Axial_DIN0204_L3.6mm_D1.6mm_P1.90mm_Vertical" V 6630 4250 50  0001 C CNN
 F 3 "~" H 6700 4250 50  0001 C CNN
 	1    6700 4250
@@
 F 0 "R6" H 7120 2096 50  0000 L CNN
 F 1 "R" H 7120 2005 50  0000 L CNN
-F 2 "" V 6980 2050 50  0001 C CNN
+F 2 "Resistor_THT:R_Axial_DIN0204_L3.6mm_D1.6mm_P1.90mm_Vertical" V 6980 2050 50  0001 C CNN
 F 3 "~" H 7050 2050 50  0001 C CNN
 	1    7050 2050
@@
 	1    0    0    -1
 $EndComp
-Text GLabel 8900 3600 2    50   Input ~ 0
+Text GLabel 8900 3450 2    50   Input ~ 0
 VIN
 $Comp
@@
 F 0 "R4" V 6393 2400 50  0000 C CNN
 F 1 "R" V 6484 2400 50  0000 C CNN
-F 2 "" V 6530 2400 50  0001 C CNN
+F 2 "Resistor_THT:R_Axial_DIN0204_L3.6mm_D1.6mm_P1.90mm_Vertical" V 6530 2400 50  0001 C CNN
 F 3 "~" H 6600 2400 50  0001 C CNN
 	1    6600 2400
@@
 F 0 "R5" H 6820 2096 50  0000 L CNN
 F 1 "R" H 6820 2005 50  0000 L CNN
-F 2 "" V 6680 2050 50  0001 C CNN
+F 2 "Resistor_THT:R_Axial_DIN0204_L3.6mm_D1.6mm_P1.90mm_Vertical" V 6680 2050 50  0001 C CNN
 F 3 "~" H 6750 2050 50  0001 C CNN
 	1    6750 2050
@@
 Text GLabel 9350 2950 0    50   Input ~ 0
 DAT
-Text GLabel 4650 3500 2    50   Input ~ 0
+Text GLabel 4700 3500 2    50   Input ~ 0
 ALFA
-Text GLabel 4650 3600 2    50   Input ~ 0
+Text GLabel 4700 3600 2    50   Input ~ 0
 BETA
 Text GLabel 4650 3900 2    50   Input ~ 0
@@
 L power:VCC #PWR0112
 U 1 1 606F8E0E
-P 4050 3200
-F 0 "#PWR0112" H 4050 3050 50  0001 C CNN
-F 1 "VCC" H 4067 3373 50  0000 C CNN
-F 2 "" H 4050 3200 50  0001 C CNN
-F 3 "" H 4050 3200 50  0001 C CNN
-	1    4050 3200
+P 4050 3100
+F 0 "#PWR0112" H 4050 2950 50  0001 C CNN
+F 1 "VCC" H 4067 3273 50  0000 C CNN
+F 2 "" H 4050 3100 50  0001 C CNN
+F 3 "" H 4050 3100 50  0001 C CNN
+	1    4050 3100
 	1    0    0    -1
 $EndComp
@@
 L power:GND #PWR0113
 U 1 1 606F8EC7
-P 4050 4400
-F 0 "#PWR0113" H 4050 4150 50  0001 C CNN
-F 1 "GND" H 4055 4227 50  0000 C CNN
-F 2 "" H 4050 4400 50  0001 C CNN
-F 3 "" H 4050 4400 50  0001 C CNN
-	1    4050 4400
+P 4050 4500
+F 0 "#PWR0113" H 4050 4250 50  0001 C CNN
+F 1 "GND" H 4055 4327 50  0000 C CNN
+F 2 "" H 4050 4500 50  0001 C CNN
+F 3 "" H 4050 4500 50  0001 C CNN
+	1    4050 4500
 	1    0    0    -1
 $EndComp
@@
 F 0 "C1" H 1165 2246 50  0000 L CNN
 F 1 "C" H 1165 2155 50  0000 L CNN
-F 2 "" H 1088 2050 50  0001 C CNN
+F 2 "Capacitor_THT:CP_Axial_L10.0mm_D6.0mm_P15.00mm_Horizontal" H 1088 2050 50  0001 C CNN
 F 3 "~" H 1050 2200 50  0001 C CNN
 	1    1050 2200
@@
 F 0 "C2" H 1815 2246 50  0000 L CNN
 F 1 "C" H 1815 2155 50  0000 L CNN
-F 2 "" H 1738 2050 50  0001 C CNN
+F 2 "Capacitor_THT:CP_Axial_L10.0mm_D6.0mm_P15.00mm_Horizontal" H 1738 2050 50  0001 C CNN
 F 3 "~" H 1700 2200 50  0001 C CNN
 	1    1700 2200
@@
 L power:VCC #PWR0117
 U 1 1 606F94BE
-P 1700 2050
-F 0 "#PWR0117" H 1700 1900 50  0001 C CNN
-F 1 "VCC" H 1717 2223 50  0000 C CNN
-F 2 "" H 1700 2050 50  0001 C CNN
-F 3 "" H 1700 2050 50  0001 C CNN
-	1    1700 2050
+P 1700 1900
+F 0 "#PWR0117" H 1700 1750 50  0001 C CNN
+F 1 "VCC" H 1717 2073 50  0000 C CNN
+F 2 "" H 1700 1900 50  0001 C CNN
+F 3 "" H 1700 1900 50  0001 C CNN
+	1    1700 1900
 	1    0    0    -1
 $EndComp
@@
 L power:GND #PWR0119
 U 1 1 606F9B37
-P 8900 3700
-F 0 "#PWR0119" H 8900 3450 50  0001 C CNN
-F 1 "GND" V 8905 3572 50  0000 R CNN
-F 2 "" H 8900 3700 50  0001 C CNN
-F 3 "" H 8900 3700 50  0001 C CNN
-	1    8900 3700
+P 8800 3700
+F 0 "#PWR0119" H 8800 3450 50  0001 C CNN
+F 1 "GND" V 8805 3572 50  0000 R CNN
+F 2 "" H 8800 3700 50  0001 C CNN
+F 3 "" H 8800 3700 50  0001 C CNN
+	1    8800 3700
 	0    1    1    0
 $EndComp
@@
 Wire Wire Line
 	7050 1900 7050 1750
+Wire Wire Line
+	8800 3450 8900 3450
+Wire Wire Line
+	8800 3700 8900 3700
+Wire Wire Line
+	4050 4400 4050 4500
+Wire Wire Line
+	4650 3500 4700 3500
+Wire Wire Line
+	4650 3600 4700 3600
+Wire Wire Line
+	4050 3100 4050 3200
+Wire Wire Line
+	1700 1900 1700 2050
+$Comp
+L Connector_Generic_MountingPin:Conn_01x08_MountingPin J5
+U 1 1 607A075A
+P 8900 5600
+F 0 "J5" H 8987 5516 50  0000 L CNN
+F 1 "Conn_01x08_MountingPin" H 8987 5425 50  0000 L CNN
+F 2 "Connector_PinHeader_2.54mm:PinHeader_1x08_P2.54mm_Vertical" H 8900 5600 50  0001 C CNN
+F 3 "~" H 8900 5600 50  0001 C CNN
+	1    8900 5600
+	1    0    0    -1
+$EndComp
+Text GLabel 8450 5300 0    50   Input ~ 0
+VIN
+Text GLabel 8450 5400 0    50   Input ~ 0
+GND
+Text GLabel 8450 5500 0    50   Input ~ 0
+O5V
+Text GLabel 8450 5600 0    50   Input ~ 0
+GND
+Text GLabel 8450 5700 0    50   Input ~ 0
+O3V
+Text GLabel 8450 5800 0    50   Input ~ 0
+GND
+Text GLabel 8450 5900 0    50   Input ~ 0
+CLK
+Text GLabel 8450 6000 0    50   Input ~ 0
+DAT
+Wire Wire Line
+	8450 5300 8700 5300
+Wire Wire Line
+	8450 5400 8700 5400
+Wire Wire Line
+	8450 5500 8700 5500
+Wire Wire Line
+	8450 5600 8700 5600
+Wire Wire Line
+	8450 5700 8700 5700
+Wire Wire Line
+	8450 5800 8700 5800
+Wire Wire Line
+	8450 5900 8700 5900
+Wire Wire Line
+	8450 6000 8700 6000
 $EndSCHEMATC

Commit message: Aktualizacja schematu.
Parts:
- removed J1: VOUT 3V, Connector_PinHeader_2.54mm:PinHeader_1x01_P2.54mm_Horizontal, symbol Connector:Conn_01x02_Male
- removed J2: Power IN, Connector_PinHeader_2.54mm:PinHeader_1x01_P2.54mm_Horizontal, symbol Connector:Conn_01x02_Male
- removed J3: I2C, Connector_PinHeader_2.54mm:PinHeader_1x01_P2.54mm_Horizontal, symbol Connector:Conn_01x02_Male
- removed J4: VOUT 5V, Connector_PinHeader_2.54mm:PinHeader_1x01_P2.54mm_Horizontal, symbol Connector:Conn_01x02_Male
- removed Q1, Q3: IRF4905, Package_TO_SOT_THT:TO-220-3_Vertical, symbol Transistor_FET:IRF4905
- removed Q4: 2N2219, Package_TO_SOT_THT:TO-39-3, symbol Transistor_BJT:2N2219
- removed R2, R4, R5, R6: R, Resistor_THT:R_Axial_DIN0204_L3.6mm_D1.6mm_P1.90mm_Vertical, symbol Device:R
- added D?: LED, symbol Device:LED
- added Q?: IRF9540N, Package_TO_SOT_THT:TO-220-3_Vertical, symbol Transistor_FET:IRF9540N
- added R?: 330, symbol Device:R
- Q2: value 2N2219 -> BC547C
- R1: value R -> 1k
- R3: value R -> 100k
Connections:
- net +5V: now also R3.1, Q?.3 (S); no longer J5.1 (Pin_1)
- net ALFA: now also U1.2 (XTAL1/PB3); no longer U1.5 (AREF/PB0)
- net CLK: no longer U1.3 (XTAL2/PB4)
- net DAT: no longer U1.2 (XTAL1/PB3)
- net GND: now also R?.2; no longer U1.1 (~RESET~/PB5), U1.7 (PB2)
- net O3V: now also Q?.2 (D)
- net VCC: no longer R3.1
- net at Q2.3 (C), R3.2: now also Q?.1 (G)
- net BETA: no longer names the net of U1.6 (PB1)
- net BETA: now also D?.2 (A)
- new net: D?.1 (K), R?.1
- new net VIN: J5.1 (Pin_1)
Other:
- moved on the sheet: R3
